Commit message: updated modle to be more realistic

File: urdf/robocam.urdf (robot description, URDF)
Before this commit: robot robocam, 7 links, 6 joints
Links:
- added link link_f1; visual cylinder length=.07 radius=0.03
- added link link_f2; visual cylinder length=.05 radius=0.03
- link base: geometry visual cylinder length=.08 radius=0.03
- link link_1: geometry visual cylinder length=.32 radius=0.03
- link link_2: geometry visual cylinder length=.32 radius=0.03
- link link_pitch: geometry visual cylinder length=.05 radius=0.03
- link link_roll: geometry visual cylinder length=.02 radius=0.03
- link link_rot: geometry visual cylinder length=.04 radius=0.03
- link link_yaw: geometry visual cylinder length=.02 radius=0.02
Joints:
- removed joint joint_1_2
- removed joint joint_2_pitch
- added joint joint_1_f1: type fixed, parent link_1, child link_f1, origin xyz=0 0 .32 rpy=-0.4720 0 0
- added joint joint_2_f2: type fixed, parent link_2, child link_f2, origin xyz=0 0 .32 rpy=-1.1139 0 0
- added joint joint_f1_2: type continuous, parent link_f1, child link_2, origin xyz=0 0 .04 rpy=0 0 0, axis 1 0 0
- added joint joint_f2_pitch: type continuous, parent link_f2, child link_pitch, origin xyz=0 0 0.05 rpy=-.5163 0 0, axis 1 0 0
- joint joint_base_rot: origin xyz=0 0 .5 rpy=0 0 0 -> xyz=0 0 .08 rpy=0 0 0
- joint joint_pitch_yaw: axis 0 1 0 -> 0 0 1; origin xyz=0 0 .5 rpy=0 0 0 -> xyz=0 0.0225 .05 rpy=0 0 0
- joint joint_rot_1: origin xyz=0 0 .5 rpy=0 0 0 -> xyz=0 0 .04 rpy=-0.2507 0 0
- joint joint_yaw_roll: origin xyz=0 0 .5 rpy=0 0 0 -> xyz=0 0 0.05 rpy=0 1.57 0

Commit message: more realistic urdf with joint limits

File: urdf/robocam.urdf (robot description, URDF)
Before this commit: robot robocam, 9 links, 8 joints
Links:
- added link link_camera; visual cylinder length=.002 radius=0.02
- link base: geometry visual cylinder length=.065 radius=0.03
- link link_f1: geometry visual cylinder length=.058 radius=0.039
- link link_f2: geometry visual cylinder length=.0656 radius=0.03
- link link_pitch: geometry visual cylinder length=.051 radius=0.0196
- link link_roll: geometry visual box size=0.04588 0.04588 0.003
- link link_rot: geometry visual cylinder length=.05 radius=0.03
- link link_yaw: geometry visual cylinder length=.02475 radius=0.01996
Joints:
- added joint joint_roll_camera: type fixed, parent link_roll, child link_camera, origin xyz=0 0 -.003 rpy=0 0 0
- joint joint_1_f1: origin xyz=0 0 .32 rpy=-0.4720 0 0 -> xyz=0 0 .32 rpy=-0.5470 0 0
- joint joint_2_f2: origin xyz=0 0 .32 rpy=-1.1139 0 0 -> xyz=0 0.0168 .32 rpy=0.4672 0 0
- joint joint_base_rot: limit (none) -> lower=-1.57 upper=1.57 effort=1000.0 velocity=1000; origin xyz=0 0 .08 rpy=0 0 0 -> xyz=0 0 .065 rpy=0 0 0; type continuous -> revolute
- joint joint_f1_2: limit (none) -> lower=-.3927 upper=.3927 effort=1000.0 velocity=1000; origin xyz=0 0 .04 rpy=0 0 0 -> xyz=0 0.0117 0.0374 rpy=-1.57 0 0; type continuous -> revolute
- joint joint_f2_pitch: limit (none) -> lower=-1.57 upper=1.57 effort=1000.0 velocity=1000; origin xyz=0 0 0.05 rpy=-.5163 0 0 -> xyz=0 0 0.0603 rpy=-.4672 0 0; type continuous -> revolute
- joint joint_pitch_yaw: limit (none) -> lower=-1.57 upper=1.57 effort=1000.0 velocity=1000; origin xyz=0 0.0225 .05 rpy=0 0 0 -> xyz=0 -0.0196 .038655 rpy=1.57 0 0; type continuous -> revolute
- joint joint_rot_1: limit (none) -> lower=-.3927 upper=0.3927 effort=1000.0 velocity=1000; origin xyz=0 0 .04 rpy=-0.2507 0 0 -> xyz=0 0.013 .05 rpy=0 0 0; type continuous -> revolute
- joint joint_yaw_roll: limit (none) -> lower=-1.57 upper=1.57 effort=1000.0 velocity=1000; origin xyz=0 0 0.05 rpy=0 1.57 0 -> xyz=0 0.02182 0.01582 rpy=1.57 0 0; type continuous -> revolute

Commit message: added dummy inertial values and collision boxes

File: urdf/robocam.urdf (robot description, URDF)
Before this commit: robot robocam, 10 links, 9 joints
Links:
- link base: mass None -> .6; geometry collision cylinder length=.065 radius=0.03; visual cylinder length=.065 radius=0.03
- link link_1: mass None -> 1.5; geometry collision cylinder length=.32 radius=0.03; visual cylinder length=.32 radius=0.03
- link link_2: mass None -> 1.5; geometry collision cylinder length=.32 radius=0.03; visual cylinder length=.32 radius=0.03
- link link_camera: mass None -> .2; geometry collision cylinder length=.002 radius=0.02; visual cylinder length=.002 radius=0.02
- link link_f1: mass None -> .8; geometry collision cylinder length=.058 radius=0.039; visual cylinder length=.058 radius=0.039
- link link_f2: mass None -> .8; geometry collision cylinder length=.0656 radius=0.03; visual cylinder length=.0656 radius=0.03
- link link_pitch: mass None -> .2; geometry collision cylinder length=.051 radius=0.0196; visual cylinder length=.051 radius=0.0196
- link link_roll: mass None -> .2; geometry collision box size=0.04588 0.04588 0.003; visual box size=0.04588 0.04588 0.003
- link link_rot: mass None -> .6; geometry collision cylinder length=.05 radius=0.03; visual cylinder length=.05 radius=0.03
- link link_yaw: mass None -> .2; geometry collision cylinder length=.02475 radius=0.01996; visual cylinder length=.02475 radius=0.01996

Commit message: changed to parallelogram

File: urdf/robocam.urdf (robot description, URDF)
Before this commit: robot robocam, 10 links, 9 joints
Links:
- added link link_1_mimic, mass 1.5; collision cylinder length=.32 radius=0.005; visual cylinder length=.32 radius=0.005
- added link link_2_mimic, mass 1.5; collision cylinder length=.32 radius=0.005; visual cylinder length=.32 radius=0.005
- link link_1: geometry collision cylinder length=.32 radius=0.005; visual cylinder length=.32 radius=0.005
- link link_2: geometry collision cylinder length=.32 radius=0.005; visual cylinder length=.32 radius=0.005
- link link_f1: geometry collision cylinder length=.06 radius=0.039; visual cylinder length=.06 radius=0.039
- link link_f2: geometry collision cylinder length=.07 radius=0.03; visual cylinder length=.07 radius=0.03
- link link_rot: geometry collision cylinder length=.06 radius=0.03; visual cylinder length=.06 radius=0.03
Joints:
- added joint joint_1_mimic_f1: type continuous, parent link_1_mimic, child link_f1, origin xyz=0 0 .32 rpy=-0.5470 0 0, mimic joint=joint_rot_1 multiplier=-1 offset=0
- added joint joint_2_mimic_f2: type continuous, parent link_2_mimic, child link_f2, origin xyz=0 0 .32 rpy=0.4672 0 0, mimic joint=joint_f1_2 multiplier=-1 offset=0
- added joint joint_f1_2_mimic: type continuous, parent link_f1, child link_2_mimic, origin xyz=0 0.02 0.0174 rpy=-1.57 0 0, axis 1 0 0, mimic joint=joint_f1_2 multiplier=1 offset=0
- added joint joint_rot_1_mimic: type revolute, parent link_rot, child link_1_mimic, origin xyz=0 -0.01 .07 rpy=0 0 0, axis 1 0 0, limit lower=-.3927 upper=0.3927 effort=1000.0 velocity=1000, mimic joint=joint_rot_1 multiplier=1 offset=0
- joint joint_2_f2: origin xyz=0 0.0168 .32 rpy=0.4672 0 0 -> xyz=0 0 .32 rpy=0.4672 0 0
- joint joint_f1_2: origin xyz=0 0.0117 0.0374 rpy=-1.57 0 0 -> xyz=0 0 0.0374 rpy=-1.57 0 0
- joint joint_rot_1: origin xyz=0 0.013 .05 rpy=0 0 0 -> xyz=0 0.01 .05 rpy=0 0 0

Commit message: updated urdf with longer links

File: urdf/robocam.urdf (robot description, URDF)
Before this commit: robot robocam, 12 links, 13 joints
Links:
- link link_1: geometry collision cylinder length=.342 radius=0.005; visual cylinder length=.342 radius=0.005
- link link_1_mimic: geometry collision cylinder length=.342 radius=0.005; visual cylinder length=.342 radius=0.005
- link link_2: geometry collision cylinder length=.34 radius=0.005; visual cylinder length=.34 radius=0.005
- link link_2_mimic: geometry collision cylinder length=.34 radius=0.005; visual cylinder length=.34 radius=0.005

Commit message: updated urdf with longer links and adjusted joint positions

File: urdf/robocam.urdf (robot description, URDF)
Before this commit: robot robocam, 12 links, 13 joints
Links:
- link link_1: geometry collision cylinder length=.336 radius=0.005; visual cylinder length=.336 radius=0.005
- link link_1_mimic: geometry collision cylinder length=.336 radius=0.005; visual cylinder length=.336 radius=0.005
Joints:
- joint joint_1_f1: origin xyz=0 0 .32 rpy=-0.5470 0 0 -> xyz=0 0 .337 rpy=-0.5470 0 0
- joint joint_1_mimic_f1: origin xyz=0 0 .32 rpy=-0.5470 0 0 -> xyz=0 0 .337 rpy=-0.5470 0 0
- joint joint_2_f2: origin xyz=0 0 .32 rpy=0.4672 0 0 -> xyz=0 0 .34 rpy=0.4672 0 0
- joint joint_2_mimic_f2: origin xyz=0 0 .32 rpy=0.4672 0 0 -> xyz=0 0 .34 rpy=0.4672 0 0

Commit message: updated values so more closely align with KDL links

File: urdf/robocam.urdf (robot description, URDF)
Before this commit: robot robocam, 12 links, 13 joints
Links:
- link base: geometry collision cylinder length=.083 radius=0.03; visual cylinder length=.083 radius=0.03
- link link_camera: geometry collision cylinder length=.02 radius=0.02; visual cylinder length=.005 radius=0.02
- link link_roll: geometry collision box size=0.04588 0.04588 0.007; visual box size=0.04588 0.04588 0.007
- link link_rot: geometry collision cylinder length=.083 radius=0.03; visual cylinder length=.083 radius=0.03
Joints:
- joint joint_1_f1: origin xyz=0 0 .337 rpy=-0.5470 0 0 -> xyz=0 0 .336 rpy=-0.5470 0 0
- joint joint_1_mimic_f1: origin xyz=0 0 .337 rpy=-0.5470 0 0 -> xyz=0 0 .336 rpy=-0.5470 0 0
- joint joint_base_rot: origin xyz=0 0 .065 rpy=0 0 0 -> xyz=0 -.032 .083 rpy=0 0 0
- joint joint_f2_pitch: origin xyz=0 0 0.0603 rpy=-.4672 0 0 -> xyz=0 0 0.0464 rpy=-.4672 0 0
- joint joint_pitch_yaw: origin xyz=0 -0.0196 .038655 rpy=1.57 0 0 -> xyz=0 -0.013 .039 rpy=1.57 0 0
- joint joint_roll_camera: origin xyz=0 0 -.003 rpy=0 0 0 -> xyz=0 0.024 .008 rpy=0 0 0
- joint joint_rot_1: origin xyz=0 0.01 .05 rpy=0 0 0 -> xyz=0 0.012 .041 rpy=0 0 0
- joint joint_rot_1_mimic: origin xyz=0 -0.01 .07 rpy=0 0 0 -> xyz=0 -0.012 .07 rpy=0 0 0
- joint joint_yaw_roll: origin xyz=0 0.02182 0.01582 rpy=1.57 0 0 -> xyz=0 0.021 0.017 rpy=1.57 0 0

Commit message: updated base offset

File: urdf/robocam.urdf (robot description, URDF)
Before this commit: robot robocam, 12 links, 13 joints
Links:
- link base: geometry collision cylinder length=.07 radius=0.03; visual cylinder length=.07 radius=0.03
- link link_rot: geometry collision cylinder length=.07 radius=0.03; visual cylinder length=.07 radius=0.03
Joints:
- joint joint_base_rot: origin xyz=0 -.032 .083 rpy=0 0 0 -> xyz=0 -.032 .07 rpy=0 0 0

Commit message: Update robocam.urdf

File: urdf/robocam.urdf (robot description, URDF)
Before this commit: robot robocam, 12 links, 13 joints
Links:
- link base: mass .6 -> None
Joints:
- removed joint joint_1_mimic_f1
- removed joint joint_2_mimic_f2
- joint joint_1_f1: axis (none) -> 1 0 0; mimic (none) -> joint=joint_rot_1 multiplier=-1 offset=0; type fixed -> continuous
- joint joint_2_f2: axis (none) -> 1 0 0; mimic (none) -> joint=joint_f1_2 multiplier=-1 offset=0; origin xyz=0 0 .34 rpy=0.4672 0 0 -> xyz=0 0.34 0 rpy=0 0 0; type fixed -> continuous
- joint joint_base_rot: origin xyz=0 -.032 .07 rpy=0 0 0 -> xyz=0 0 .07 rpy=0 0 0
- joint joint_f1_2: origin xyz=0 0 0.0374 rpy=-1.57 0 0 -> xyz=0 0 0.0374 rpy=0 0 0
- joint joint_f1_2_mimic: origin xyz=0 0.02 0.0174 rpy=-1.57 0 0 -> xyz=0 0.02 0.0174 rpy=0 0 0
- joint joint_f2_pitch: origin xyz=0 0 0.0464 rpy=-.4672 0 0 -> xyz=0 0.0464 0 rpy=0 0 0
- joint joint_pitch_yaw: origin xyz=0 -0.013 .039 rpy=1.57 0 0 -> xyz=0 0.039 0.013 rpy=0 0 0
- joint joint_roll_camera: origin xyz=0 0.024 .008 rpy=0 0 0 -> xyz=0 0.008 0.024 rpy=0 0 0
- joint joint_yaw_roll: axis 0 0 1 -> 0 1 0; origin xyz=0 0.021 0.017 rpy=1.57 0 0 -> xyz=0 0.021 0.017 rpy=0 0 0

Commit message: Update robocam.urdf

File: urdf/robocam.urdf (robot description, URDF)
Before this commit: robot robocam, 12 links, 11 joints
Joints:
- joint joint_roll_camera: origin xyz=0 0.008 0.024 rpy=0 0 0 -> xyz=0 0.0177 0.0063 rpy=0 0 0
- joint joint_yaw_roll: origin xyz=0 0.021 0.017 rpy=0 0 0 -> xyz=0.005 0.023 0.016 rpy=0 0 0
